Commit message: feat: integrate H2 real-stand retraining baseline

File: assets/urdf/h2_description/H2_stand.urdf (robot description, URDF)
Before this commit: robot H2_stand, 37 links, 36 joints
Joints:
- joint left_ankle_pitch_joint: limit lower=-1.059842014 upper=0.685487238 effort=66.88 velocity=28.61 -> lower=-1.13446401358 upper=0.61086523808 effort=66.88 velocity=28.61; origin xyz=-0.014516 -0.0373 0 rpy=0 -0.074622000 0 -> xyz=-0.014516 -0.0373 0 rpy=0 0 0
- joint left_ankle_roll_joint: limit lower=-0.326720850 upper=0.319050973 effort=19 velocity=100.7 -> lower=-0.3490658503 upper=0.296705972783 effort=19 velocity=100.7; origin xyz=0.032719 -0.023002 -0.49662 rpy=-0.022345000 0 0 -> xyz=0.032719 -0.023002 -0.49662 rpy=0 0 0
- joint left_elbow_joint: origin xyz=0.016655 0.02211 -0.12792 rpy=0 0 0 -> xyz=0.016655 0.02211 -0.12792 rpy=0 1.1 0
- joint left_hip_pitch_joint: limit lower=-2.506969500 upper=2.721050500 effort=360 velocity=20 -> lower=-2.4525975 upper=2.7754225 effort=360 velocity=20; origin xyz=0 0.08038 -0.046407 rpy=-0.524240614 0.047081695 -0.027206165 -> xyz=0 0.08038 -0.046407 rpy=-0.5236 0 0
- joint left_hip_roll_joint: limit lower=-0.523521000 upper=2.112780500 effort=360 velocity=20 -> lower=-0.467441 upper=2.1688605 effort=360 velocity=20; origin xyz=0.041774 0.0635 -0.019 rpy=0.579680000 0 0 -> xyz=0.041774 0.0635 -0.019 rpy=0.5236 0 0
- joint left_hip_yaw_joint: limit lower=-3.041685000 upper=2.612315000 effort=360 velocity=20 -> lower=-2.827 upper=2.827 effort=360 velocity=20; origin xyz=-0.028187 -0.0095 -0.0737 rpy=0 0 0.214685000 -> xyz=-0.028187 -0.0095 -0.0737 rpy=0 0 0
- joint left_knee_joint: limit lower=-0.172697000 upper=2.444803000 effort=360 velocity=20 -> lower=-0.08725 upper=2.53025 effort=360 velocity=20; origin xyz=-0.010308 0.022549 -0.31959 rpy=0 0.085447000 0 -> xyz=-0.010308 0.022549 -0.31959 rpy=0 0 0
- joint left_shoulder_roll_joint: origin xyz=-0.0032074 0.059938 -0.039865 rpy=-0.26914 0 0 -> xyz=-0.0032074 0.059938 -0.039865 rpy=0.13086 0 0
- joint left_shoulder_yaw_joint: origin xyz=-0.0025601 0.0036752 -0.10421 rpy=0 0 0 -> xyz=-0.0025601 0.0036752 -0.10421 rpy=0 0 -0.4
- joint right_ankle_pitch_joint: limit lower=-1.067509014 upper=0.677820238 effort=66.88 velocity=28.61 -> lower=-1.13446401358 upper=0.61086523808 effort=66.88 velocity=28.61; origin xyz=-0.014516 0.0373 0 rpy=0 -0.066955000 0 -> xyz=-0.014516 0.0373 0 rpy=0 0 0
- joint right_ankle_roll_joint: limit lower=-0.356322973 upper=0.289448850 effort=19 velocity=100.7 -> lower=-0.296705972783 upper=0.3490658503 effort=19 velocity=100.7; origin xyz=0.032719 0.023002 -0.49662 rpy=0.059617000 0 0 -> xyz=0.032719 0.023002 -0.49662 rpy=0 0 0
- joint right_elbow_joint: origin xyz=0.016655 -0.02211 -0.12792 rpy=0 0 0 -> xyz=0.016655 -0.02211 -0.12792 rpy=0 1.1 0
- joint right_hip_pitch_joint: limit lower=-2.524442500 upper=2.703577500 effort=360 velocity=20 -> lower=-2.4525975 upper=2.7754225 effort=360 velocity=20; origin xyz=0 -0.08038 -0.046407 rpy=0.524719228 0.062206150 0.035968991 -> xyz=0 -0.08038 -0.046407 rpy=0.5236 0 0
- joint right_hip_roll_joint: limit lower=-2.112430500 upper=0.523871000 effort=360 velocity=20 -> lower=-2.1688605 upper=0.467441 effort=360 velocity=20; origin xyz=0.041774 -0.0635 -0.019 rpy=-0.580030000 0 0 -> xyz=0.041774 -0.0635 -0.019 rpy=-0.5236 0 0
- joint right_hip_yaw_joint: limit lower=-2.705004000 upper=2.948996000 effort=360 velocity=20 -> lower=-2.827 upper=2.827 effort=360 velocity=20; origin xyz=-0.028187 0.0095 -0.0737 rpy=0 0 -0.121996000 -> xyz=-0.028187 0.0095 -0.0737 rpy=0 0 0
- joint right_knee_joint: limit lower=-0.201614000 upper=2.415886000 effort=360 velocity=20 -> lower=-0.08725 upper=2.53025 effort=360 velocity=20; origin xyz=-0.010308 -0.022549 -0.31959 rpy=0 0.114364000 0 -> xyz=-0.010308 -0.022549 -0.31959 rpy=0 0 0
- joint right_shoulder_roll_joint: origin xyz=-0.0032074 -0.059938 -0.039865 rpy=0.26914 0 0 -> xyz=-0.0032074 -0.059938 -0.039865 rpy=-0.13086 0 0
- joint right_shoulder_yaw_joint: origin xyz=-0.0025601 -0.0036752 -0.10421 rpy=0 0 0 -> xyz=-0.0025601 -0.0036752 -0.10421 rpy=0 0 0.4
